Commit message: added odom transform

File: src/dead/urdf/robot.urdf (robot description, URDF)
Before this commit: robot Dead_wheelrobot, 4 links, 3 joints
Links:
- link base_link: geometry visual box size=0.186 0.255 0.1

Commit message: updated

File: src/dead/urdf/robot.urdf (robot description, URDF)
Before this commit: robot Dead_wheelrobot, 4 links, 3 joints
Links:
- link deadwheel_x_one: geometry visual cylinder length=0.0125 radius=0.0295
- link deadwheel_x_two: geometry visual cylinder length=0.0125 radius=0.0295
- link deadwheel_y_one: geometry visual cylinder length=0.0125 radius=0.0295
Joints:
- joint deadwheel_x_left: origin xyz=0.0 -0.0965 -0.05 rpy=0 0 0 -> xyz=0.093 -0.1275 -0.0795 rpy=0 0 0
- joint deadwheel_x_right: origin xyz=0.0 0.0965 -0.05 rpy=0 0 0 -> xyz=0.093 0.1275 -0.0795 rpy=0 0 0
- joint deadwheel_y: origin xyz=-0.065 0.0 -0.05 rpy=0 0 0 -> xyz=-0.093 0 -0.0795 rpy=0 0 0
